File: Lotus 46 unWired/PCB v1.00/Dongle.kicad_sch (KiCad schematic)
At the start: 30 parts, among them J1 Conn_01x02, J2 Conn_01x02, J3 Conn_01x01, J4 Conn_01x01, U1 nRF52810-QCxx

Commit message: Test
Parts:
- removed C3: 1.5pF, Capacitor_SMD:C_0402_1005Metric, symbol Device:C_Small
- removed C3: 0.8pF, Capacitor_SMD:C_0402_1005Metric, symbol Device:C_Small
- removed L1 (x2): 3.9nH, Inductor_SMD:L_0402_1005Metric, symbol Device:L_Small
- removed U1: nRF52810-QCxx, Package_DFN_QFN:QFN-32-1EP_5x5mm_P0.5mm_EP3.6x3.6mm_ThermalVias, symbol MCU_Nordic:nRF52810-QCxx
- added C3: 1.5pF, Capacitor_SMD:C_0402_1005Metric, symbol Device:C_Small
- added C3: 0.8pF, Capacitor_SMD:C_0402_1005Metric, symbol Device:C_Small
- added L1 (x2): 3.9nH, Inductor_SMD:L_0402_1005Metric, symbol Device:L_Small
- added U3: nRF52810-QCxx, Package_DFN_QFN:QFN-32-1EP_5x5mm_P0.5mm_EP3.6x3.6mm_ThermalVias, symbol MCU_Nordic:nRF52810-QCxx
- C1, C2: LCSC (none) -> C458856
- C10: LCSC (none) -> C5137572
- C4, C5, C8: LCSC (none) -> C126523
- C6: value NC -> DNP; now left out of the parts list
- C7: LCSC (none) -> C147476
- C9: LCSC (none) -> C380326
- E1: LCSC (none) -> C2917722
- J1, J2: footprint Connector_PinHeader_2.54mm:PinHeader_1x02_P2.54mm_Vertical -> Keyboard Common:Pinheader_2; now left out of the parts list
- J3, J4: footprint Connector_PinHeader_2.54mm:PinHeader_1x01_P2.54mm_Vertical -> Keyboard Common:PinHeader_1; now left out of the parts list
- LED1: LCSC C965799 -> C2286
- LED2: LCSC C965805 -> C72043
- R1, R2: LCSC (none) -> C162901
- TP1, TP2, TP3, TP4: now left out of the parts list
- Y1: value ~ -> 7F32000E08UCG; LCSC (none) -> C524692
Connections:
- net +3V3: now also U3.25 (VDD), U3.32 (VDD), U3.9 (VDD)
- net GND: now also C3.1, L1.1, U3.20 (VSS), U3.29 (VSS), U3.33 (VSS)
- net SCL: now also U3.3 (P0.01/XL2)
- net SDA: now also U3.2 (P0.00/XL1)
- net SWDCLK: now also U3.17 (SWDCLK)
- net SWDIO: now also U3.18 (SWDIO)
- net at C2.2, Y1.3: now also U3.23 (XC1)
- net at E1.1: now also C3.2, L1.2
- net at LED1.2 (A): now also U3.26 (P0.25)
- net at C10.2: now also U3.30 (DEC4), U3.31 (DCC)
- net at PAIR1.2: now also U3.28 (P0.30/AIN6)
- net at C1.1, Y1.1: now also U3.24 (XC2)
- net at C4.2: now also U3.1 (DEC1)
- net at C6.2: now also U3.21 (DEC2)
- net at LED2.2 (A): now also U3.27 (P0.28/AIN4)
- net at C7.2: now also U3.22 (DEC3)
- new net: C3.1, L1.1
- new net: C3.2, L1.2, U3.19 (ANT)
Other:
- company: Tweety's Wild Thinking -> (none)
- title: unWired Dongle RP2040 -> (none)
