File: unWired Dongle RP2040/v1.00/unWired Dongle RP2040.kicad_pcb (KiCad board)
At the start: 2 copper layers, 18 x 28.4 mm, 30 parts, among them J1 Conn_01x02, J2 Conn_01x02, J3 Conn_01x01, J4 Conn_01x01, U1 nRF52810-QCxx

Commit message: Test
Parts:
- renumbered RES1 to PAIR1
Connections:
- net SCL renamed /SCL
- net SDA renamed /SDA
- net SWCLK renamed /SWDCLK
- net SWDIO renamed /SWDIO
