File: Lotus 46 unWired/Plate v1.00/Lotus46_unWired_Plate_100.kicad_sch (KiCad schematic)
At the start: 0 parts

Commit message: Cleanup plate
Parts:
- added SW1, SW10, SW11, SW12, SW13, SW14, SW15, SW16, SW17, SW18, SW2, SW20, SW21, SW22, SW23, SW3, SW4, SW5, SW6, SW7, SW8, SW9: Switch, Keyboard_Plate:SW_MX_Plate_Placeholder_nodrill_NOBORDER, symbol Switch:SW_Push
- added SW19: Switch, Keyboard_Plate:SW_MX_Plate_Placeholder_nodrill_NOBORDER, symbol Keyboard Switches:SW_Push_GND
- added TH1, TH2, TH3, TH4: HOLE, Keyboard_Plate:Spacer Plate hole, symbol keebio:Hole
Connections:
- new net SW1: SW1.1
- new net SW10: SW10.1
- new net SW11: SW11.1
- new net SW12: SW12.1
- new net SW13: SW13.1
- new net SW14: SW14.1
- new net SW15: SW15.1
- new net SW16: SW16.1
- new net SW17: SW17.1
- new net SW18: SW18.1
- new net SW19: SW19.2
- new net SW2: SW2.1
- new net SW20: SW20.1
- new net SW21: SW21.1
- new net SW22: SW22.1
- new net SW23: SW23.1
- new net SW3: SW3.1
- new net SW4: SW4.1
- new net SW5: SW5.1
- new net SW6: SW6.1
- new net SW7: SW7.1
- new net SW8: SW8.1
- new net SW9: SW9.1
Other:
- removed sheet Right Matrix
